File: HV_HBridge.sch (KiCad schematic (older format))
At the start: 28 parts, among them U1 IR2104

Commit message: first update
Parts:
- added R5, R6, R7, R8: R_Small, Resistor_THT:R_Axial_DIN0309_L9.0mm_D3.2mm_P5.08mm_Vertical, symbol Device:R_Small
- Q1: renamed from Q?; footprint (none) -> Package_TO_SOT_SMD:TO-263-2; MFN (none) -> 747-IXTA02N250HV
- Q2, Q3, Q4: renamed from Q?; footprint (none) -> Package_TO_SOT_SMD:TO-263-2
- gave numbers to parts that had none: 21
Connections:
- net GND: now also D5.2 (A), D7.2 (A); no longer D5.1 (K), D7.1 (K)
- net LOAD1: now also D4.2 (A), D5.1 (K); no longer D4.1 (K), D5.2 (A)
- net LOAD2: now also D6.2 (A), D7.1 (K); no longer D6.1 (K), D7.2 (A)
- net VCC: now also D4.1 (K), D6.1 (K); no longer D4.2 (A), D6.2 (A)
- new net: R5.2, R6.1
- new net: R6.2, R7.1
- new net: R7.2, R8.1

Commit message: updated to latest version
Parts:
- removed C1, C2, C3, C4, C5, C6, C7, C8: C_Small, symbol Device:C_Small
- removed D1: D_Schottky_Small, HV_HBridge:FM2500, symbol Device:D_Schottky_Small
- removed D10, D4, D5, D6, D7: FM2500, HV_HBridge:FM2500, symbol Device:D_Schottky_Small
- removed D2, D3, D8, D9: D_Small, symbol Device:D_Small
- removed Q1, Q2, Q3, Q4: BSS127, Package_TO_SOT_SMD:TO-263-2, symbol Device:Q_NMOS_GSD
- removed R1, R2, R3, R4: R_Small, symbol Device:R_Small
- removed R5, R6, R7, R8: R_Small, Resistor_THT:R_Axial_DIN0309_L9.0mm_D3.2mm_P5.08mm_Vertical, symbol Device:R_Small
- removed U1, U2: IR2104, symbol Driver_FET:IR2104
Other:
- note removed: "HBridge"
- note removed: "HBridge1"
- note removed: "PWM1_Driver"
